Commit message: resolvendo problema no xacro

File: ros2_ws/install/manipulator3/share/manipulator3/urdf/cores.xacro (robot description, xacro)
@@ -1,23 +1,12 @@
 <?xml version="1.0"?>
 <robot name = "manipulador" xmlns:xacro="http://www.ros.org/wiki/xacro" >
-    <!-- Cor Vermelha -->
-    <material name="red">
-        <color rgba="0.8 0 0 1"/>
+    <material name="black">
+        <color rgba="0.0 0.0 0.0 1.0"/>
     </material>
-    <!-- Cor Verde -->
-    <material name="green">
-        <color rgba="0 0.8 0 1"/>
+    <material name="white">
+        <color rgba="1.0 1.0 1.0 1.0"/>
     </material>
-    <!-- Cor Azul -->
     <material name="blue">
-        <color rgba="0 0 0.8 1"/>
-    </material>
-    <!-- Cor Amarela -->
-    <material name="yellow">
-        <color rgba="1 1 0 1"/>
-    </material>
-    <!-- Cor Ciano -->
-    <material name="cyan">
-        <color rgba="0 1 1 1"/>
+        <color rgba="0.0 0.0 0.5 1.0"/>
     </material>
 </robot>

File: ros2_ws/install/manipulator3/share/manipulator3/urdf/manipulator3.urdf.xacro (robot description, xacro)
@@ -8,4 +8,9 @@
     <xacro:property name="effort"   value="1000" />
     <xacro:property name="velocity" value="0.5" />
+    <gazebo>
+        <plugin name="gazebo_ros_control" filename="libgazebo_ros_control.so">
+            <robotNamespace>/</robotNamespace>
+        </plugin>
+    </gazebo>
     <xacro:macro name="joint_limits">
         <limit
@@ -15,25 +20,4 @@
             upper="${upper}" />
     </xacro:macro>
-    <!-- Carregar arquivo YAML -->
-    <xacro:property name="yaml_file" value="$(find manipulator3)/config/link2_inertia.yaml" />
-    <xacro:property name="link2_inertia" value="${xacro.load_yaml(yaml_file)}" />
-    <!-- manipulador description.-->
-    <!-- Link: world-->
-    <link name="world">
-        <visual>
-            <geometry>
-                <box size="0.0 0.0 0.0"/>
-            </geometry>
-            <origin rpy="0 0 0" xyz="0 0 0"/>
-            <material name="green"/>
-        </visual>
-    </link>
-    <!-- Joint 0: world para vertical1-->
-    <joint name="joint_0" type="fixed">
-        <parent link="world"/>
-        <child link="vertical1"/>
-        <origin xyz="0 0 0.23"
-                rpy="0 0 0"/>
-    </joint>
     <!-- Link 1: vertical1-->
     <link name="vertical1">
@@ -55,5 +39,5 @@
             <origin xyz="0 0 0"
                     rpy="1.5708 0 0" />
-            <material name="green"/>
+            <material name="black"/>
         </visual>
         <collision>
@@ -95,5 +79,5 @@
             <origin xyz="0 0 0"
                     rpy="1.5708 0 0" />
-            <material name="green"/>
+            <material name="blue"/>
         </visual>
         <collision>
@@ -133,5 +117,5 @@
             <origin xyz="0 0 -35"
                     rpy="1.5708 0 0" />
-            <material name="red"/>
+            <material name="white"/>
         </visual>
         <collision>
@@ -173,5 +157,5 @@
             <origin xyz="-65 0 -35"
                     rpy="1.5708 0 0" />
-            <material name="yellow"/>
+            <material name="black"/>
         </visual>
         <collision>
@@ -251,5 +235,5 @@
             <origin xyz="-27 0 0"
                     rpy="1.5708 0 3.1415" />
-            <material name="cyan"/>
+            <material name="white"/>
         </visual>
         <collision>

File: ros2_ws/src/manipulator3/install/manipulator3/share/manipulator3/urdf/manipulator3.urdf.xacro (robot description, xacro)
@@ -20,4 +20,21 @@
             upper="${upper}" />
     </xacro:macro>
+    <!-- Link: world-->
+    <link name="world">
+        <visual>
+            <geometry>
+                <box size="0.0 0.0 0.0"/>
+            </geometry>
+            <origin rpy="0 0 0" xyz="0 0 0"/>
+            <material name="green"/>
+        </visual>
+    </link>
+    <!-- Joint 0: world para vertical1-->
+    <joint name="joint_0" type="fixed">
+        <parent link="world"/>
+        <child link="vertical1"/>
+        <origin xyz="0 0 0.23"
+                rpy="0 0 0"/>
+    </joint>
     <!-- Link 1: vertical1-->
     <link name="vertical1">
